Commit message: fix dynamixel down by adding a link at the same place as the joint. updated right leg to use the new down.

File: dog_picker_description/urdf/dog_picker_leg.xacro (robot description, xacro)
@@ -9,7 +9,16 @@
       <child link="dynamixel_AX12_${dyn1}_link"/>
     </joint>
-    <xacro:dynamixel_AX12_down child="dynamixel_AX12_${dyn2}_link" number="${dyn1}" x_loc="${-AX12_Z_CENTER*2-AX12_Z_SIZE}" y_loc="${-F7_Z_SIZE+-AX12_X_SIZE/2}" z_loc="${-AX12_Z_CENTER}" r="${-90*M_PI/180} " p="0" y="${90*M_PI/180}"/>
-    <!--rotate back-->
-    <xacro:dynamixel_AX12_down child="calf_link_${dyn3}" number="${dyn2}" x_loc="0" y_loc="${F2_Y_CENTER}" z_loc="${AX12_Z_SIZE+2*AX12_Z_CENTER}" r="0" p="0" y="0"/>
+    <xacro:dynamixel_AX12_down number="${dyn1}" x_loc="0" y_loc="0" z_loc="0" r="0" p="0" y="0"/>
+    <joint name="S1_${dyn1}" type="fixed">
+      <origin xyz="${-AX12_Z_SIZE-2*AX12_Z_CENTER} ${-AX12_X_SIZE/2 - F7_Z_SIZE}  ${AX12_Y_CENTER}" rpy="${-90*M_PI/180} 0 ${90*M_PI/180} "/>
+      <parent link="S-B_${dyn1}_link"/>
+      <child link="dynamixel_AX12_${dyn2}_link"/>
+    </joint>
+    <xacro:dynamixel_AX12_down number="${dyn2}" x_loc="0" y_loc="0" z_loc="0" r="0" p="0"  y="0"/>
+      <joint name="S1_${dyn2}" type="fixed">
+      <origin xyz="0 ${F2_Y_CENTER} ${F2_Z_SIZE-F2_Z_CENTER}" rpy="0 0 0"/>
+      <parent link="S-B_${dyn2}_link"/>
+      <child link="calf_link_${dyn3}"/>
+    </joint>
     <link name="calf_link_${dyn3}">
       <visual>

File: dynamixel_description/urdf/AX12.xacro (robot description, xacro)
@@ -40,10 +40,10 @@
     </link>
   </xacro:macro>
-  <xacro:macro name="dynamixel_AX12_down" params="child number x_loc y_loc z_loc r p y">
+  <xacro:macro name="dynamixel_AX12_down" params="number x_loc y_loc z_loc r p y">
     <link name="dynamixel_AX12_${number}_link">
       <!---rviz -->
       <visual>
         <!--link origin is a delta from the joint to the center of the servo box-->
-        <origin xyz="0 ${AX12_Y_CENTER} ${AX12_Z_CENTER}" rpy="0 0 0"/>
+        <origin xyz="${x_loc} ${y_loc+AX12_Y_CENTER} ${z_loc+AX12_Z_CENTER}" rpy="0 0 0"/>
         <geometry>
           <!-- <mesh filename="package://pi_tb_description/meshes/ax12_box.${MESH_EXT}" scale="${M_SCALE} ${M_SCALE} ${M_SCALE}"/> -->
@@ -58,10 +58,21 @@
     <joint name="dynamixel_AX12_${number}_joint" type="revolute">
       <!--origin of whole dynamixel is at the center of the round part visible on the servo which is the joint -->
-      <origin xyz="${x_loc} ${y_loc} ${z_loc}" rpy="${r} ${p} ${y}"/>
+           <origin xyz="${x_loc} ${y_loc} ${z_loc}" rpy="0 0 0"/>
       <axis xyz="0 -1 0"/>
       <limit effort="${AX12_EFFORT}" lower="${-150*M_PI/180}" upper="${150*M_PI/180}" velocity="${AX12_VELOCITY}"/>
       <parent link="dynamixel_AX12_${number}_link"/>
-      <child link="${child}"/>
+      <child link="S-B_${number}_link"/>
     </joint>
+     <link name="S-B_${number}_link">
+        <visual>
+        <origin xyz="0 0 0" rpy="0 0 0"/>
+       <geometry>
+          <sphere radius="0.004"/>
+        </geometry>
+        <material name="Green">
+          <color rgba="0 0.5 0 1.0"/>
+        </material>
+      </visual>
+    </link>
   </xacro:macro>
 </robot>

Commit message: dynamixel_up with extra joint and visual

File: dog_picker_description/urdf/dog_picker_leg.xacro (robot description, xacro)
@@ -10,4 +10,5 @@
     </joint>
     <xacro:dynamixel_AX12_down number="${dyn1}" x_loc="0" y_loc="0" z_loc="0" r="0" p="0" y="0"/>
+    <!-- this fixed joint is really just placing the revolute joint in the next ax12 that way I can just always pass 0 to ax12-->
     <joint name="S1_${dyn1}" type="fixed">
       <origin xyz="${-AX12_Z_SIZE-2*AX12_Z_CENTER} ${-AX12_X_SIZE/2 - F7_Z_SIZE}  ${AX12_Y_CENTER}" rpy="${-90*M_PI/180} 0 ${90*M_PI/180} "/>
@@ -32,5 +33,10 @@
       </visual>
     </link>
-    <xacro:dynamixel_AX12_up parent="calf_link_${dyn3}" number="${dyn3}" x_loc="0" y_loc="${-F2_Y_CENTER}" z_loc="${AX12_Z_SIZE+2*AX12_Z_CENTER}" r="0" p="${180*M_PI/180} " y="0"/>
+      <joint name="S1_${dyn3}" type="fixed">
+      <origin xyz="0 ${-F2_Y_CENTER} ${F2_Z_SIZE-F2_Z_CENTER}" rpy="0 ${180*M_PI/180} 0"/>
+      <parent link="calf_link_${dyn3}"/>
+      <child link="S-B_${dyn3}_link"/>
+    </joint>
+    <xacro:dynamixel_AX12_up number="${dyn3}" x_loc="0" y_loc="0" z_loc="0" r="0" p="0" y="0"/>
   </xacro:macro>
   <xacro:macro name="dog_picker_leg_left" params="parent dyn1 dyn2 dyn3 x_loc y_loc z_loc r p y back">

File: dynamixel_description/urdf/AX12.xacro (robot description, xacro)
@@ -2,6 +2,17 @@
 <robot xmlns:xacro="http://www.ros.org/wiki/xacro" name="dynamixel">
   <xacro:include filename="$(find dynamixel_description)/urdf/constants.xacro"/>
-  <xacro:macro name="dynamixel_AX12_up" params="parent number x_loc y_loc z_loc r p y">
+  <xacro:macro name="dynamixel_AX12_up" params="number x_loc y_loc z_loc r p y">
     <!---Kinematics for kdl tree and robot_state_publisher -->
+         <link name="S-B_${number}_link">
+        <visual>
+        <origin xyz="0 0 0" rpy="0 0 0"/>
+       <geometry>
+          <sphere radius="${S_B_RADIUS}"/>
+        </geometry>
+        <material name="Green">
+          <color rgba="0 0.5 0 1.0"/>
+        </material>
+      </visual>
+    </link>
     <joint name="dynamixel_AX12_${number}_joint" type="revolute">
       <!--origin of whole dynamixel is at the center of the round part visible on the servo which is the joint -->
@@ -10,5 +21,5 @@
       <axis xyz="0 -1 0"/>
       <limit effort="${AX12_EFFORT}" lower="${-150*M_PI/180}" upper="${150*M_PI/180}" velocity="${AX12_VELOCITY}"/>
-      <parent link="${parent}"/>
+      <parent link="S-B_${number}_link"/>
       <child link="dynamixel_AX12_${number}_link"/>
     </joint>
@@ -68,5 +79,5 @@
         <origin xyz="0 0 0" rpy="0 0 0"/>
        <geometry>
-          <sphere radius="0.004"/>
+          <sphere radius="${S_B_RADIUS}"/>
         </geometry>
         <material name="Green">

File: dynamixel_description/urdf/constants.xacro (robot description, xacro)
@@ -38,3 +38,4 @@
   <xacro:property name="ACM5_Y_SIZE" value="0.100"/>
   <xacro:property name="ACM5_Z_SIZE" value="0.032"/>
+  <xacro:property name="S_B_RADIUS" value="0.004"/>
 </robot>

Commit message: left leg fix with extra joints

File: dog_picker_description/urdf/dog_picker_leg.xacro (robot description, xacro)
@@ -46,7 +46,17 @@
       <child link="dynamixel_AX12_${dyn1}_link"/>
     </joint>
-    <xacro:dynamixel_AX12_down child="dynamixel_AX12_${dyn2}_link" number="${dyn1}" x_loc="${AX12_Z_CENTER*2+AX12_Z_SIZE}" y_loc="${-F7_Z_SIZE+-AX12_X_SIZE/2}" z_loc="${-AX12_Z_CENTER}" r="${-90*M_PI/180}" p="0" y="${-90*M_PI/180}"/>
-    <!--rotate back-->
-    <xacro:dynamixel_AX12_down child="calf_link_${dyn3}" number="${dyn2}" x_loc="0" y_loc="${F2_Y_CENTER}" z_loc="${AX12_Z_SIZE+2*AX12_Z_CENTER}" r="0" p="0" y="0"/>
+      <xacro:dynamixel_AX12_down number="${dyn1}" x_loc="0" y_loc="0" z_loc="0" r="0" p="0" y="0"/>
+    <!-- this fixed joint is really just placing the revolute joint in the next ax12 that way I can just always pass 0 to ax12-->
+    <joint name="S1_${dyn1}" type="fixed">
+      <origin xyz="${AX12_Z_SIZE+2*AX12_Z_CENTER} ${-AX12_X_SIZE/2 - F7_Z_SIZE}  ${AX12_Y_CENTER}" rpy="${-90*M_PI/180} 0 ${-90*M_PI/180} "/>
+      <parent link="S-B_${dyn1}_link"/>
+      <child link="dynamixel_AX12_${dyn2}_link"/>
+    </joint>
+    <xacro:dynamixel_AX12_down number="${dyn2}" x_loc="0" y_loc="0" z_loc="0" r="0" p="0"  y="0"/>
+      <joint name="S1_${dyn2}" type="fixed">
+      <origin xyz="0 ${F2_Y_CENTER} ${F2_Z_SIZE-F2_Z_CENTER}" rpy="0 0 0"/>
+      <parent link="S-B_${dyn2}_link"/>
+      <child link="calf_link_${dyn3}"/>
+    </joint>
     <link name="calf_link_${dyn3}">
       <visual>
@@ -60,5 +70,10 @@
       </visual>
     </link>
-    <xacro:dynamixel_AX12_up parent="calf_link_${dyn3}" number="${dyn3}" x_loc="0" y_loc="${-F2_Y_CENTER}" z_loc="${AX12_Z_SIZE+2*AX12_Z_CENTER}" r="0" p="${180*M_PI/180} " y="0"/>
+      <joint name="S1_${dyn3}" type="fixed">
+      <origin xyz="0 ${-F2_Y_CENTER} ${F2_Z_SIZE-F2_Z_CENTER}" rpy="0 ${180*M_PI/180} 0"/>
+      <parent link="calf_link_${dyn3}"/>
+      <child link="S-B_${dyn3}_link"/>
+    </joint>
+    <xacro:dynamixel_AX12_up number="${dyn3}" x_loc="0" y_loc="0" z_loc="0" r="0" p="0" y="0"/>
   </xacro:macro>
 </robot>
