Commit message: dog picker finished with new fixed joints in appropiate places

File: dog_picker_description/urdf/dog_picker_description.xacro (robot description, xacro)
@@ -33,6 +33,16 @@
     </visual>
   </link>
-  <xacro:dynamixel_AX12_up parent="neck_link" number="6" x_loc="${F3_Z_SIZE+F1_Z_SIZE/2 +F1_Z_CENTER}" y_loc="${F1_Y_CENTER}" z_loc="${F1_X_SIZE/2-ACM5_Z_SIZE/2+F1_X_CENTER}" r="${M_PI} " p="0 " y="0"/>
-  <xacro:dynamixel_AX12_up parent="dynamixel_AX12_6_link" number="17" x_loc="0" y_loc="${AX12_Y_CENTER}" z_loc="${-AX12_Z_SIZE-AX12_Z_CENTER - F3_Z_SIZE}" r="${-90*M_PI/180}" p="0" y="${90*M_PI/180}"/>
+  <joint name="S1_6" type="fixed">
+      <origin xyz="${F3_Z_SIZE+F1_Z_SIZE/2 +F1_Z_CENTER} ${F1_Y_CENTER} ${F1_X_SIZE/2-ACM5_Z_SIZE/2+F1_X_CENTER}" rpy="${M_PI} 0 0"/>
+      <parent link="neck_link"/>
+      <child link="S-B_6_link"/>
+    </joint>
+  <xacro:dynamixel_AX12_up number="6" x_loc="0" y_loc="0" z_loc="0" r="0" p="0 " y="0"/>
+  <joint name="S1_17" type="fixed">
+      <origin xyz="0 ${AX12_Y_CENTER} ${-AX12_Z_SIZE-AX12_Z_CENTER - F3_Z_SIZE}" rpy="${-90*M_PI/180} 0 ${90*M_PI/180}"/>
+      <parent link="dynamixel_AX12_6_link"/>
+      <child link="S-B_17_link"/>
+    </joint>
+  <xacro:dynamixel_AX12_up number="17" x_loc="0" y_loc="0" z_loc="0" r="0" p="0 " y="0"/>
   <joint name="robotis_part_1" type="fixed">
     <origin xyz="-0.045 0 0.150" rpy="0 0 0"/>
@@ -51,5 +61,10 @@
     </visual>
   </link>
-  <xacro:dynamixel_AX12_up parent="butt_link" number="1" x_loc="${-F2_Z_SIZE- F3_Z_SIZE+ F2_Z_CENTER} " y_loc="${-AX12_Y_CENTER}" z_loc="0" r="0" p="${90*M_PI/180}" y="0"/>
+    <joint name="S1_1" type="fixed">
+      <origin xyz="${-F2_Z_SIZE- F3_Z_SIZE+ F2_Z_CENTER} ${-AX12_Y_CENTER} 0" rpy="0 ${90*M_PI/180} 0"/>
+      <parent link="butt_link"/>
+      <child link="S-B_1_link"/>
+    </joint>
+  <xacro:dynamixel_AX12_up number="1" x_loc="0" y_loc="0" z_loc="0" r="0" p="0 " y="0"/>
   <xacro:dog_picker_leg_right parent="base_link" dyn1="4" dyn2="16" dyn3="8" x_loc="${ACM5_X_SIZE/2}" y_loc="${-ACM5_Y_SIZE/2-AX12_Z_CENTER}" z_loc="${0.150-ACM5_Z_SIZE/2-F3_Z_SIZE-F10_Z_SIZE-AX12_X_SIZE/2}" r="0" p="0 " y="0" back="0"/>
   <xacro:dog_picker_leg_right parent="dynamixel_AX12_1_link" dyn1="11" dyn2="13" dyn3="15" x_loc="${F3_Z_SIZE+F10_Z_SIZE +AX12_X_SIZE}" y_loc="${F1_Y_CENTER+AX12_Z_SIZE+AX12_Z_CENTER}" z_loc="${-AX12_Y_SIZE}" r="0" p="${90*M_PI/180}" y="0" back="1"/>

Commit message: changed physical neck and urdf to match

File: dog_picker_description/urdf/dog_picker_description.xacro (robot description, xacro)
@@ -17,35 +17,13 @@
     </visual>
   </link>
-  <joint name="robotis_part_6" type="fixed">
-    <origin xyz="${ACM5_X_SIZE/2} 0 0.150" rpy="0 0 0"/>
+  <joint name="robotis_part_3" type="fixed">
+    <origin xyz="${ACM5_X_SIZE/2 + AX12_Z_SIZE + AX12_Z_CENTER + 2*F3_Z_SIZE} 0 ${ACM5_Z_SIZE/2 + 0.150}" rpy="${-90*M_PI/180} 0 ${-90*M_PI/180} "/>
     <parent link="base_link"/>
-    <child link="neck_link"/>
+    <child link="dynamixel_AX12_3_link"/>
   </joint>
-  <link name="neck_link">
-    <visual>
-      <origin rpy="0 0 0" xyz="${(F1_Z_SIZE + F3_Z_SIZE)/2} 0 ${F1_X_SIZE/2-0.016}"/>
-      <geometry>
-        <box size="${F1_Z_SIZE + F3_Z_SIZE} ${F1_Y_SIZE}  ${F1_X_SIZE} "/>
-      </geometry>
-      <material name="DimWhite">
-        <color rgba="0.9 0.9 0.9 1.0"/>
-      </material>
-    </visual>
-  </link>
-  <joint name="S1_6" type="fixed">
-      <origin xyz="${F3_Z_SIZE+F1_Z_SIZE/2 +F1_Z_CENTER} ${F1_Y_CENTER} ${F1_X_SIZE/2-ACM5_Z_SIZE/2+F1_X_CENTER}" rpy="${M_PI} 0 0"/>
-      <parent link="neck_link"/>
-      <child link="S-B_6_link"/>
-    </joint>
-  <xacro:dynamixel_AX12_up number="6" x_loc="0" y_loc="0" z_loc="0" r="0" p="0 " y="0"/>
-  <joint name="S1_17" type="fixed">
-      <origin xyz="0 ${AX12_Y_CENTER} ${-AX12_Z_SIZE-AX12_Z_CENTER - F3_Z_SIZE}" rpy="${-90*M_PI/180} 0 ${90*M_PI/180}"/>
-      <parent link="dynamixel_AX12_6_link"/>
-      <child link="S-B_17_link"/>
-    </joint>
-  <xacro:dynamixel_AX12_up number="17" x_loc="0" y_loc="0" z_loc="0" r="0" p="0 " y="0"/>
+  <xacro:dynamixel_AX12_down number="3" x_loc="0" y_loc="0" z_loc="0" r="0" p="0 " y="0"/>
   <joint name="S1_kinect" type="fixed">
-      <origin xyz="0 ${AX12_Y_SIZE + 0.045} 0" rpy="0 0 0"/>
-      <parent link="dynamixel_AX12_17_link"/>
+      <origin xyz="0 -0.050 0" rpy="0 0 0"/>
+      <parent link="S-B_3_link"/>
       <child link="kinect_link"/>
     </joint>

Commit message: clean up xyx and rpy by setting to 0 in ax12. using joints before hand to orient ax12

File: dog_picker_description/urdf/dog_picker_description.xacro (robot description, xacro)
@@ -22,5 +22,5 @@
     <child link="dynamixel_AX12_3_link"/>
   </joint>
-  <xacro:dynamixel_AX12_down number="3" x_loc="0" y_loc="0" z_loc="0" r="0" p="0 " y="0"/>
+  <xacro:dynamixel_AX12_down number="3"/>
   <joint name="S1_kinect" type="fixed">
       <origin xyz="0 -0.050 0" rpy="0 0 0"/>
@@ -60,5 +60,5 @@
       <child link="S-B_1_link"/>
     </joint>
-  <xacro:dynamixel_AX12_up number="1" x_loc="0" y_loc="0" z_loc="0" r="0" p="0 " y="0"/>
+  <xacro:dynamixel_AX12_up number="1"/>
   <xacro:dog_picker_leg_right parent="base_link" dyn1="4" dyn2="16" dyn3="8" x_loc="${ACM5_X_SIZE/2}" y_loc="${-ACM5_Y_SIZE/2-AX12_Z_CENTER}" z_loc="${0.150-ACM5_Z_SIZE/2-F3_Z_SIZE-F10_Z_SIZE-AX12_X_SIZE/2}" r="0" p="0 " y="0" back="0"/>
   <xacro:dog_picker_leg_right parent="dynamixel_AX12_1_link" dyn1="11" dyn2="13" dyn3="15" x_loc="${F3_Z_SIZE+F10_Z_SIZE +AX12_X_SIZE}" y_loc="${F1_Y_CENTER+AX12_Z_SIZE+AX12_Z_CENTER}" z_loc="${-AX12_Y_SIZE}" r="0" p="${90*M_PI/180}" y="0" back="1"/>

File: dog_picker_description/urdf/dog_picker_leg.xacro (robot description, xacro)
@@ -9,5 +9,5 @@
       <child link="dynamixel_AX12_${dyn1}_link"/>
     </joint>
-    <xacro:dynamixel_AX12_down number="${dyn1}" x_loc="0" y_loc="0" z_loc="0" r="0" p="0" y="0"/>
+    <xacro:dynamixel_AX12_down number="${dyn1}"/>
     <!-- this fixed joint is really just placing the revolute joint in the next ax12 that way I can just always pass 0 to ax12-->
     <joint name="S1_${dyn1}" type="fixed">
@@ -16,5 +16,5 @@
       <child link="dynamixel_AX12_${dyn2}_link"/>
     </joint>
-    <xacro:dynamixel_AX12_down number="${dyn2}" x_loc="0" y_loc="0" z_loc="0" r="0" p="0"  y="0"/>
+    <xacro:dynamixel_AX12_down number="${dyn2}"/>
       <joint name="S1_${dyn2}" type="fixed">
       <origin xyz="0 ${F2_Y_CENTER} ${F2_Z_SIZE-F2_Z_CENTER}" rpy="0 0 0"/>
@@ -38,5 +38,5 @@
       <child link="S-B_${dyn3}_link"/>
     </joint>
-    <xacro:dynamixel_AX12_up number="${dyn3}" x_loc="0" y_loc="0" z_loc="0" r="0" p="0" y="0"/>
+    <xacro:dynamixel_AX12_up number="${dyn3}"/>
   </xacro:macro>
   <xacro:macro name="dog_picker_leg_left" params="parent dyn1 dyn2 dyn3 x_loc y_loc z_loc r p y back">
@@ -46,5 +46,5 @@
       <child link="dynamixel_AX12_${dyn1}_link"/>
     </joint>
-      <xacro:dynamixel_AX12_down number="${dyn1}" x_loc="0" y_loc="0" z_loc="0" r="0" p="0" y="0"/>
+      <xacro:dynamixel_AX12_down number="${dyn1}"/>
     <!-- this fixed joint is really just placing the revolute joint in the next ax12 that way I can just always pass 0 to ax12-->
     <joint name="S1_${dyn1}" type="fixed">
@@ -53,5 +53,5 @@
       <child link="dynamixel_AX12_${dyn2}_link"/>
     </joint>
-    <xacro:dynamixel_AX12_down number="${dyn2}" x_loc="0" y_loc="0" z_loc="0" r="0" p="0"  y="0"/>
+    <xacro:dynamixel_AX12_down number="${dyn2}"/>
       <joint name="S1_${dyn2}" type="fixed">
       <origin xyz="0 ${F2_Y_CENTER} ${F2_Z_SIZE-F2_Z_CENTER}" rpy="0 0 0"/>
@@ -75,5 +75,5 @@
       <child link="S-B_${dyn3}_link"/>
     </joint>
-    <xacro:dynamixel_AX12_up number="${dyn3}" x_loc="0" y_loc="0" z_loc="0" r="0" p="0" y="0"/>
+    <xacro:dynamixel_AX12_up number="${dyn3}"/>
   </xacro:macro>
 </robot>

File: dynamixel_description/urdf/AX12.xacro (robot description, xacro)
@@ -2,5 +2,5 @@
 <robot xmlns:xacro="http://www.ros.org/wiki/xacro" name="dynamixel">
   <xacro:include filename="$(find dynamixel_description)/urdf/constants.xacro"/>
-  <xacro:macro name="dynamixel_AX12_up" params="number x_loc y_loc z_loc r p y">
+  <xacro:macro name="dynamixel_AX12_up" params="number">
     <!---Kinematics for kdl tree and robot_state_publisher -->
          <link name="S-B_${number}_link">
@@ -17,5 +17,5 @@
     <joint name="dynamixel_AX12_${number}_joint" type="revolute">
       <!--origin of whole dynamixel is at the center of the round part visible on the servo which is the joint -->
-      <origin xyz="${x_loc} ${y_loc} ${z_loc}" rpy="${r} ${p} ${y}"/>
+      <origin xyz="0 0 0" rpy="0 0 0"/>
       <!-- negative green is the joint axis... -->
       <axis xyz="0 -1 0"/>
@@ -51,10 +51,10 @@
     </link>
   </xacro:macro>
-  <xacro:macro name="dynamixel_AX12_down" params="number x_loc y_loc z_loc r p y">
+  <xacro:macro name="dynamixel_AX12_down" params="number">
     <link name="dynamixel_AX12_${number}_link">
       <!---rviz -->
       <visual>
         <!--link origin is a delta from the joint to the center of the servo box-->
-        <origin xyz="${x_loc} ${y_loc+AX12_Y_CENTER} ${z_loc+AX12_Z_CENTER}" rpy="0 0 0"/>
+        <origin xyz="0 ${0+AX12_Y_CENTER} ${0+AX12_Z_CENTER}" rpy="0 0 0"/>
         <geometry>
           <!-- <mesh filename="package://pi_tb_description/meshes/ax12_box.${MESH_EXT}" scale="${M_SCALE} ${M_SCALE} ${M_SCALE}"/> -->
@@ -69,5 +69,5 @@
     <joint name="dynamixel_AX12_${number}_joint" type="revolute">
       <!--origin of whole dynamixel is at the center of the round part visible on the servo which is the joint -->
-           <origin xyz="${x_loc} ${y_loc} ${z_loc}" rpy="0 0 0"/>
+           <origin xyz="0 0 0" rpy="0 0 0"/>
       <axis xyz="0 -1 0"/>
       <limit effort="${AX12_EFFORT}" lower="${-150*M_PI/180}" upper="${150*M_PI/180}" velocity="${AX12_VELOCITY}"/>
