Commit message: update dog.urdf and test a moveit setup

File: dog_picker_description/urdf/dog.urdf (robot description, URDF)
Before this commit: robot dog_picker, 22 links, 21 joints
Links:
- added link S-B_10_link; visual sphere radius=0.004
- added link S-B_11_link; visual sphere radius=0.004
- added link S-B_12_link; visual sphere radius=0.004
- added link S-B_13_link; visual sphere radius=0.004
- added link S-B_14_link; visual sphere radius=0.004
- added link S-B_15_link; visual sphere radius=0.004
- added link S-B_16_link; visual sphere radius=0.004
- added link S-B_17_link; visual sphere radius=0.004
- added link S-B_1_link; visual sphere radius=0.004
- added link S-B_4_link; visual sphere radius=0.004
- added link S-B_5_link; visual sphere radius=0.004
- added link S-B_6_link; visual sphere radius=0.004
- added link S-B_7_link; visual sphere radius=0.004
- added link S-B_8_link; visual sphere radius=0.004
- added link S-B_9_link; visual sphere radius=0.004
Joints:
- added joint S1_1: type fixed, parent butt_link, child S-B_1_link, origin xyz=-0.0355 -0.02 0 rpy=0 1.570795 0
- added joint S1_10: type fixed, parent S-B_10_link, child dynamixel_AX12_12_link, origin xyz=0.023 -0.021  0.02 rpy=-1.570795 0 -1.570795 
- added joint S1_11: type fixed, parent S-B_11_link, child dynamixel_AX12_13_link, origin xyz=-0.023 -0.021  0.02 rpy=-1.570795 0 1.570795 
- added joint S1_12: type fixed, parent S-B_12_link, child calf_link_14, origin xyz=0 0.021 0.0305 rpy=0 0 0
- added joint S1_13: type fixed, parent S-B_13_link, child calf_link_15, origin xyz=0 0.021 0.0305 rpy=0 0 0
- added joint S1_14: type fixed, parent calf_link_14, child S-B_14_link, origin xyz=0 -0.021 0.0305 rpy=0 3.14159 0
- added joint S1_15: type fixed, parent calf_link_15, child S-B_15_link, origin xyz=0 -0.021 0.0305 rpy=0 3.14159 0
- added joint S1_16: type fixed, parent S-B_16_link, child calf_link_8, origin xyz=0 0.021 0.0305 rpy=0 0 0
- added joint S1_17: type fixed, parent dynamixel_AX12_6_link, child S-B_17_link, origin xyz=0 0.02 -0.0415 rpy=-1.570795 0 1.570795
- added joint S1_4: type fixed, parent S-B_4_link, child dynamixel_AX12_16_link, origin xyz=-0.023 -0.021  0.02 rpy=-1.570795 0 1.570795 
- added joint S1_5: type fixed, parent S-B_5_link, child dynamixel_AX12_7_link, origin xyz=0.023 -0.021  0.02 rpy=-1.570795 0 -1.570795 
- added joint S1_6: type fixed, parent neck_link, child S-B_6_link, origin xyz=0.027 0.021 0.0125 rpy=3.14159 0 0
- added joint S1_7: type fixed, parent S-B_7_link, child calf_link_9, origin xyz=0 0.021 0.0305 rpy=0 0 0
- added joint S1_8: type fixed, parent calf_link_8, child S-B_8_link, origin xyz=0 -0.021 0.0305 rpy=0 3.14159 0
- added joint S1_9: type fixed, parent calf_link_9, child S-B_9_link, origin xyz=0 -0.021 0.0305 rpy=0 3.14159 0
- joint dynamixel_AX12_10_joint: child dynamixel_AX12_12_link -> S-B_10_link; origin xyz=0.023 -0.021 0.0135 rpy=-1.570795 0 -1.570795 -> xyz=0 0 0 rpy=0 0 0
- joint dynamixel_AX12_11_joint: child dynamixel_AX12_13_link -> S-B_11_link; origin xyz=-0.023 -0.021 0.0135 rpy=-1.570795 0 1.570795 -> xyz=0 0 0 rpy=0 0 0
- joint dynamixel_AX12_12_joint: child calf_link_14 -> S-B_12_link; origin xyz=0 0.021 0.023 rpy=0 0 0 -> xyz=0 0 0 rpy=0 0 0
- joint dynamixel_AX12_13_joint: child calf_link_15 -> S-B_13_link; origin xyz=0 0.021 0.023 rpy=0 0 0 -> xyz=0 0 0 rpy=0 0 0
- joint dynamixel_AX12_14_joint: origin xyz=0 -0.021 0.023 rpy=0 3.14159 0 -> xyz=0 0 0 rpy=0 0 0; parent calf_link_14 -> S-B_14_link
- joint dynamixel_AX12_15_joint: origin xyz=0 -0.021 0.023 rpy=0 3.14159 0 -> xyz=0 0 0 rpy=0 0 0; parent calf_link_15 -> S-B_15_link
- joint dynamixel_AX12_16_joint: child calf_link_8 -> S-B_16_link; origin xyz=0 0.021 0.023 rpy=0 0 0 -> xyz=0 0 0 rpy=0 0 0
- joint dynamixel_AX12_17_joint: origin xyz=0 0.02 -0.0415 rpy=-1.570795 0 1.570795 -> xyz=0 0 0 rpy=0 0 0; parent dynamixel_AX12_6_link -> S-B_17_link
- joint dynamixel_AX12_1_joint: origin xyz=-0.0355 -0.02 0 rpy=0 1.570795 0 -> xyz=0 0 0 rpy=0 0 0; parent butt_link -> S-B_1_link
- joint dynamixel_AX12_4_joint: child dynamixel_AX12_16_link -> S-B_4_link; origin xyz=-0.023 -0.021 0.0135 rpy=-1.570795 0 1.570795 -> xyz=0 0 0 rpy=0 0 0
- joint dynamixel_AX12_5_joint: axis 1 0 0 -> 0 -1 0; child dynamixel_AX12_7_link -> S-B_5_link; origin xyz=0.023 -0.021 0.0135 rpy=-1.570795 0 -1.570795 -> xyz=0 0 0 rpy=0 0 0
- joint dynamixel_AX12_6_joint: origin xyz=0.027 0.021 0.0125 rpy=3.14159 0 0 -> xyz=0 0 0 rpy=0 0 0; parent neck_link -> S-B_6_link
- joint dynamixel_AX12_7_joint: child calf_link_9 -> S-B_7_link; origin xyz=0 0.021 0.023 rpy=0 0 0 -> xyz=0 0 0 rpy=0 0 0
- joint dynamixel_AX12_8_joint: origin xyz=0 -0.021 0.023 rpy=0 3.14159 0 -> xyz=0 0 0 rpy=0 0 0; parent calf_link_8 -> S-B_8_link
- joint dynamixel_AX12_9_joint: origin xyz=0 -0.021 0.023 rpy=0 3.14159 0 -> xyz=0 0 0 rpy=0 0 0; parent calf_link_9 -> S-B_9_link

Commit message: kinect link added

File: dog_picker_description/urdf/dog.urdf (robot description, URDF)
Before this commit: robot dog_picker, 37 links, 36 joints
Links:
- added link kinect_link; visual box size=0.300 0.090 0.080
Joints:
- added joint S1_kinect: type fixed, parent dynamixel_AX12_17_link, child kinect_link, origin xyz=0 0.085 0 rpy=0 0 0

File: dog_picker_description/urdf/dog_picker_description.xacro (robot description, xacro)
@@ -45,4 +45,20 @@
     </joint>
   <xacro:dynamixel_AX12_up number="17" x_loc="0" y_loc="0" z_loc="0" r="0" p="0 " y="0"/>
+  <joint name="S1_kinect" type="fixed">
+      <origin xyz="0 ${AX12_Y_SIZE + 0.045} 0" rpy="0 0 0"/>
+      <parent link="dynamixel_AX12_17_link"/>
+      <child link="kinect_link"/>
+    </joint>
+  <link name="kinect_link">
+    <visual>
+      <origin rpy="0 0 0" xyz="0 0 0"/>
+      <geometry>
+        <box size="0.300 0.090 0.080"/>
+      </geometry>
+      <material name="Blue">
+        <color rgba="0.0 0.0 0.9 1.0"/>
+      </material>
+    </visual>
+  </link>
   <joint name="robotis_part_1" type="fixed">
     <origin xyz="-0.045 0 0.150" rpy="0 0 0"/>

Commit message: updated description and added yaml params for whole connected robot

File: dog_picker_description/urdf/dog.urdf (robot description, URDF)
Before this commit: robot dog_picker, 38 links, 37 joints
Links:
- removed link S-B_17_link
- removed link S-B_6_link
- removed link dynamixel_AX12_17_link
- removed link dynamixel_AX12_6_link
- removed link neck_link
- added link S-B_3_link; visual sphere radius=0.004
- added link dynamixel_AX12_3_link; visual box size=0.032 0.04 0.05
Joints:
- removed joint S1_17
- removed joint S1_6
- removed joint dynamixel_AX12_17_joint
- removed joint dynamixel_AX12_6_joint
- removed joint robotis_part_6
- added joint dynamixel_AX12_3_joint: type revolute, parent dynamixel_AX12_3_link, child S-B_3_link, origin xyz=0 0 0 rpy=0 0 0, axis 0 -1 0, limit lower=-2.61799166667 upper=2.61799166667 effort=1000 velocity=0.5
- added joint robotis_part_3: type fixed, parent base_link, child dynamixel_AX12_3_link, origin xyz=0.0915 0 0.166 rpy=-1.570795 0 -1.570795 
- joint S1_kinect: origin xyz=0 0.085 0 rpy=0 0 0 -> xyz=0 -0.050 0 rpy=0 0 0; parent dynamixel_AX12_17_link -> S-B_3_link
